File: Keyboard Project V1/60 Percent Keyboard Project/60 Percent Keyboard Ardiuno Micro.kicad_pcb (KiCad board)
At the start: 2 copper layers, 48.3 x 17.8 mm, 6 parts, among them J1 Analog, J2 Digital

Commit message: updated version of version 1 and currently in the PCB editor. Almost done with version one and may work on version V1.1 after this
Parts:
- added A1: Arduino_Nano_v3.x, Module:Arduino_Nano, F.Cu at (254.8, 235.2)
- added D1: 1N4148, Diode_THT:D_DO-35_SOD27_P7.62mm_Horizontal, F.Cu at (5.80, 223.4)
- added D10: 1N4148, Diode_THT:D_DO-35_SOD27_P7.62mm_Horizontal, F.Cu at (41.8, 223.4)
- added D11: 1N4148, Diode_THT:D_DO-35_SOD27_P7.62mm_Horizontal, F.Cu at (45.8, 223.4)
- added D12: 1N4148, Diode_THT:D_DO-35_SOD27_P7.62mm_Horizontal, F.Cu at (49.8, 223.4)
- added D13: 1N4148, Diode_THT:D_DO-35_SOD27_P7.62mm_Horizontal, F.Cu at (53.8, 223.4)
- added D14: 1N4148, Diode_THT:D_DO-35_SOD27_P7.62mm_Horizontal, F.Cu at (57.8, 223.4)
- added D15: 1N4148, Diode_THT:D_DO-35_SOD27_P7.62mm_Horizontal, F.Cu at (61.8, 223.4)
- added D16: 1N4148, Diode_THT:D_DO-35_SOD27_P7.62mm_Horizontal, F.Cu at (65.8, 223.4)
- added D17: 1N4148, Diode_THT:D_DO-35_SOD27_P7.62mm_Horizontal, F.Cu at (69.8, 223.4)
- added D18: 1N4148, Diode_THT:D_DO-35_SOD27_P7.62mm_Horizontal, F.Cu at (73.8, 223.4)
- added D19: 1N4148, Diode_THT:D_DO-35_SOD27_P7.62mm_Horizontal, F.Cu at (77.8, 223.4)
- added D2: 1N4148, Diode_THT:D_DO-35_SOD27_P7.62mm_Horizontal, F.Cu at (9.80, 223.4)
- added D20: 1N4148, Diode_THT:D_DO-35_SOD27_P7.62mm_Horizontal, F.Cu at (81.8, 223.4)
- added D21: 1N4148, Diode_THT:D_DO-35_SOD27_P7.62mm_Horizontal, F.Cu at (85.8, 223.4)
- added D22: 1N4148, Diode_THT:D_DO-35_SOD27_P7.62mm_Horizontal, F.Cu at (89.8, 223.4)
- added D23: 1N4148, Diode_THT:D_DO-35_SOD27_P7.62mm_Horizontal, F.Cu at (93.8, 223.4)
- added D24: 1N4148, Diode_THT:D_DO-35_SOD27_P7.62mm_Horizontal, F.Cu at (97.8, 223.4)
- added D25: 1N4148, Diode_THT:D_DO-35_SOD27_P7.62mm_Horizontal, F.Cu at (101.8, 223.4)
- added D26: 1N4148, Diode_THT:D_DO-35_SOD27_P7.62mm_Horizontal, F.Cu at (105.8, 223.4)
- added D27: 1N4148, Diode_THT:D_DO-35_SOD27_P7.62mm_Horizontal, F.Cu at (109.8, 223.4)
- added D28: 1N4148, Diode_THT:D_DO-35_SOD27_P7.62mm_Horizontal, F.Cu at (113.8, 223.4)
- added D29: 1N4148, Diode_THT:D_DO-35_SOD27_P7.62mm_Horizontal, F.Cu at (117.8, 223.4)
- added D3: 1N4148, Diode_THT:D_DO-35_SOD27_P7.62mm_Horizontal, F.Cu at (13.8, 223.4)
- added D30: 1N4148, Diode_THT:D_DO-35_SOD27_P7.62mm_Horizontal, F.Cu at (121.8, 223.4)
- added D31: 1N4148, Diode_THT:D_DO-35_SOD27_P7.62mm_Horizontal, F.Cu at (125.8, 223.4)
- added D32: 1N4148, Diode_THT:D_DO-35_SOD27_P7.62mm_Horizontal, F.Cu at (129.8, 223.4)
- added D33: 1N4148, Diode_THT:D_DO-35_SOD27_P7.62mm_Horizontal, F.Cu at (133.8, 223.4)
- added D34: 1N4148, Diode_THT:D_DO-35_SOD27_P7.62mm_Horizontal, F.Cu at (137.8, 223.4)
- added D35: 1N4148, Diode_THT:D_DO-35_SOD27_P7.62mm_Horizontal, F.Cu at (141.8, 223.4)
- added D36: 1N4148, Diode_THT:D_DO-35_SOD27_P7.62mm_Horizontal, F.Cu at (145.8, 223.4)
- added D37: 1N4148, Diode_THT:D_DO-35_SOD27_P7.62mm_Horizontal, F.Cu at (149.8, 223.4)
- added D38: 1N4148, Diode_THT:D_DO-35_SOD27_P7.62mm_Horizontal, F.Cu at (153.8, 223.4)
- added D39: 1N4148, Diode_THT:D_DO-35_SOD27_P7.62mm_Horizontal, F.Cu at (157.8, 223.4)
- added D4: 1N4148, Diode_THT:D_DO-35_SOD27_P7.62mm_Horizontal, F.Cu at (17.8, 223.4)
- added D40: 1N4148, Diode_THT:D_DO-35_SOD27_P7.62mm_Horizontal, F.Cu at (161.8, 223.4)
- added D41: 1N4148, Diode_THT:D_DO-35_SOD27_P7.62mm_Horizontal, F.Cu at (165.8, 223.4)
- added D42: 1N4148, Diode_THT:D_DO-35_SOD27_P7.62mm_Horizontal, F.Cu at (169.8, 223.4)
- added D43: 1N4148, Diode_THT:D_DO-35_SOD27_P7.62mm_Horizontal, F.Cu at (173.8, 223.4)
- added D44: 1N4148, Diode_THT:D_DO-35_SOD27_P7.62mm_Horizontal, F.Cu at (177.8, 223.4)
- added D45: 1N4148, Diode_THT:D_DO-35_SOD27_P7.62mm_Horizontal, F.Cu at (181.8, 223.4)
- added D46: 1N4148, Diode_THT:D_DO-35_SOD27_P7.62mm_Horizontal, F.Cu at (185.8, 223.4)
- added D47: 1N4148, Diode_THT:D_DO-35_SOD27_P7.62mm_Horizontal, F.Cu at (189.8, 223.4)
- added D48: 1N4148, Diode_THT:D_DO-35_SOD27_P7.62mm_Horizontal, F.Cu at (193.8, 223.4)
- added D49: 1N4148, Diode_THT:D_DO-35_SOD27_P7.62mm_Horizontal, F.Cu at (197.8, 223.4)
- added D5: 1N4148, Diode_THT:D_DO-35_SOD27_P7.62mm_Horizontal, F.Cu at (21.8, 223.4)
- added D50: 1N4148, Diode_THT:D_DO-35_SOD27_P7.62mm_Horizontal, F.Cu at (201.8, 223.4)
- added D51: 1N4148, Diode_THT:D_DO-35_SOD27_P7.62mm_Horizontal, F.Cu at (205.8, 223.4)
- added D52: 1N4148, Diode_THT:D_DO-35_SOD27_P7.62mm_Horizontal, F.Cu at (209.8, 223.4)
- added D53: 1N4148, Diode_THT:D_DO-35_SOD27_P7.62mm_Horizontal, F.Cu at (213.8, 223.4)
- added D54: 1N4148, Diode_THT:D_DO-35_SOD27_P7.62mm_Horizontal, F.Cu at (217.8, 223.4)
- added D55: 1N4148, Diode_THT:D_DO-35_SOD27_P7.62mm_Horizontal, F.Cu at (221.8, 223.4)
- added D56: 1N4148, Diode_THT:D_DO-35_SOD27_P7.62mm_Horizontal, F.Cu at (225.8, 223.4)
- added D57: 1N4148, Diode_THT:D_DO-35_SOD27_P7.62mm_Horizontal, F.Cu at (229.8, 223.4)
- added D58: 1N4148, Diode_THT:D_DO-35_SOD27_P7.62mm_Horizontal, F.Cu at (233.8, 223.4)
- added D59: 1N4148, Diode_THT:D_DO-35_SOD27_P7.62mm_Horizontal, F.Cu at (237.8, 223.4)
- added D6: 1N4148, Diode_THT:D_DO-35_SOD27_P7.62mm_Horizontal, F.Cu at (25.8, 223.4)
- added D60: 1N4148, Diode_THT:D_DO-35_SOD27_P7.62mm_Horizontal, F.Cu at (241.8, 223.4)
- added D61: 1N4148, Diode_THT:D_DO-35_SOD27_P7.62mm_Horizontal, F.Cu at (245.8, 223.4)
- added D7: 1N4148, Diode_THT:D_DO-35_SOD27_P7.62mm_Horizontal, F.Cu at (29.8, 223.4)
- added D8: 1N4148, Diode_THT:D_DO-35_SOD27_P7.62mm_Horizontal, F.Cu at (33.8, 223.4)
- added D9: 1N4148, Diode_THT:D_DO-35_SOD27_P7.62mm_Horizontal, F.Cu at (37.8, 223.4)
- added MX1: MX-NoLED, Switch_Keyboard_Cherry_MX:SW_Cherry_MX_PCB_1.00u, F.Cu at (8.80, 247.7)
- added MX10: MX-NoLED, Switch_Keyboard_Cherry_MX:SW_Cherry_MX_PCB_1.25u, F.Cu at (35.8, 327.7)
- added MX11: MX-NoLED, Switch_Keyboard_Cherry_MX:SW_Cherry_MX_PCB_1.00u, F.Cu at (48.3, 247.7)
- added MX12: MX-NoLED, Switch_Keyboard_Cherry_MX:SW_Cherry_MX_PCB_1.00u, F.Cu at (58.3, 267.7)
- added MX13: MX-NoLED, Switch_Keyboard_Cherry_MX:SW_Cherry_MX_PCB_1.00u, F.Cu at (63.3, 287.7)
- added MX14: MX-NoLED, Switch_Keyboard_Cherry_MX:SW_Cherry_MX_PCB_1.00u, F.Cu at (73.3, 307.7)
- added MX15: MX-NoLED, Switch_Keyboard_Cherry_MX:SW_Cherry_MX_PCB_1.25u, F.Cu at (60.8, 327.7)
- added MX16: MX-NoLED, Switch_Keyboard_Cherry_MX:SW_Cherry_MX_PCB_1.00u, F.Cu at (68.3, 247.7)
- added MX17: MX-NoLED, Switch_Keyboard_Cherry_MX:SW_Cherry_MX_PCB_1.00u, F.Cu at (78.3, 267.7)
- added MX18: MX-NoLED, Switch_Keyboard_Cherry_MX:SW_Cherry_MX_PCB_1.00u, F.Cu at (83.3, 287.7)
- added MX19: MX-NoLED, Switch_Keyboard_Cherry_MX:SW_Cherry_MX_PCB_1.00u, F.Cu at (93.3, 307.7)
- added MX2: MX-NoLED, Switch_Keyboard_Cherry_MX:SW_Cherry_MX_PCB_1.50u, F.Cu at (13.3, 267.7)
- added MX20: MX-NoLED, Switch_Keyboard_Cherry_MX:SW_Cherry_MX_PCB_1.00u, F.Cu at (88.3, 247.7)
- added MX21: MX-NoLED, Switch_Keyboard_Cherry_MX:SW_Cherry_MX_PCB_1.00u, F.Cu at (98.3, 267.7)
- added MX22: MX-NoLED, Switch_Keyboard_Cherry_MX:SW_Cherry_MX_PCB_1.00u, F.Cu at (103.3, 287.7)
- added MX23: MX-NoLED, Switch_Keyboard_Cherry_MX:SW_Cherry_MX_PCB_1.00u, F.Cu at (113.3, 307.7)
- added MX24: MX-NoLED, Switch_Keyboard_Cherry_MX:SW_Cherry_MX_PCB_6.25u, F.Cu at (133.3, 327.7)
- added MX25: MX-NoLED, Switch_Keyboard_Cherry_MX:SW_Cherry_MX_PCB_1.00u, F.Cu at (108.3, 247.7)
- added MX26: MX-NoLED, Switch_Keyboard_Cherry_MX:SW_Cherry_MX_PCB_1.00u, F.Cu at (118.3, 267.7)
- added MX27: MX-NoLED, Switch_Keyboard_Cherry_MX:SW_Cherry_MX_PCB_1.00u, F.Cu at (123.3, 287.7)
- added MX28: MX-NoLED, Switch_Keyboard_Cherry_MX:SW_Cherry_MX_PCB_1.00u, F.Cu at (133.3, 307.7)
- added MX29: MX-NoLED, Switch_Keyboard_Cherry_MX:SW_Cherry_MX_PCB_1.00u, F.Cu at (128.3, 247.7)
- added MX3: MX-NoLED, Switch_Keyboard_Cherry_MX:SW_Cherry_MX_PCB_1.75u, F.Cu at (15.8, 287.7)
- added MX30: MX-NoLED, Switch_Keyboard_Cherry_MX:SW_Cherry_MX_PCB_1.00u, F.Cu at (138.3, 267.7)
- added MX31: MX-NoLED, Switch_Keyboard_Cherry_MX:SW_Cherry_MX_PCB_1.00u, F.Cu at (143.3, 287.7)
- added MX32: MX-NoLED, Switch_Keyboard_Cherry_MX:SW_Cherry_MX_PCB_1.00u, F.Cu at (153.3, 307.7)
- added MX33: MX-NoLED, Switch_Keyboard_Cherry_MX:SW_Cherry_MX_PCB_1.00u, F.Cu at (148.3, 247.7)
- added MX34: MX-NoLED, Switch_Keyboard_Cherry_MX:SW_Cherry_MX_PCB_1.00u, F.Cu at (158.3, 267.7)
- added MX35: MX-NoLED, Switch_Keyboard_Cherry_MX:SW_Cherry_MX_PCB_1.00u, F.Cu at (163.3, 287.7)
- added MX36: MX-NoLED, Switch_Keyboard_Cherry_MX:SW_Cherry_MX_PCB_1.00u, F.Cu at (173.3, 307.7)
- added MX37: MX-NoLED, Switch_Keyboard_Cherry_MX:SW_Cherry_MX_PCB_1.25u, F.Cu at (205.8, 327.7)
- added MX38: MX-NoLED, Switch_Keyboard_Cherry_MX:SW_Cherry_MX_PCB_1.00u, F.Cu at (168.3, 247.7)
- added MX39: MX-NoLED, Switch_Keyboard_Cherry_MX:SW_Cherry_MX_PCB_1.00u, F.Cu at (178.3, 267.7)
- added MX4: MX-NoLED, Switch_Keyboard_Cherry_MX:SW_Cherry_MX_PCB_2.25u, F.Cu at (20.8, 307.7)
- added MX40: MX-NoLED, Switch_Keyboard_Cherry_MX:SW_Cherry_MX_PCB_1.00u, F.Cu at (183.3, 287.7)
- added MX41: MX-NoLED, Switch_Keyboard_Cherry_MX:SW_Cherry_MX_PCB_1.00u, F.Cu at (193.3, 307.7)
- added MX42: MX-NoLED, Switch_Keyboard_Cherry_MX:SW_Cherry_MX_PCB_1.25u, F.Cu at (231.9, 327.8)
- added MX43: MX-NoLED, Switch_Keyboard_Cherry_MX:SW_Cherry_MX_PCB_1.00u, F.Cu at (188.3, 247.7)
- added MX44: MX-NoLED, Switch_Keyboard_Cherry_MX:SW_Cherry_MX_PCB_1.00u, F.Cu at (198.3, 267.7)
- added MX45: MX-NoLED, Switch_Keyboard_Cherry_MX:SW_Cherry_MX_PCB_1.00u, F.Cu at (203.3, 287.7)
- added MX46: MX-NoLED, Switch_Keyboard_Cherry_MX:SW_Cherry_MX_PCB_1.00u, F.Cu at (213.3, 307.7)
- added MX47: MX-NoLED, Switch_Keyboard_Cherry_MX:SW_Cherry_MX_PCB_1.25u, F.Cu at (258.4, 327.8)
- added MX48: MX-NoLED, Switch_Keyboard_Cherry_MX:SW_Cherry_MX_PCB_1.00u, F.Cu at (208.3, 247.7)
- added MX49: MX-NoLED, Switch_Keyboard_Cherry_MX:SW_Cherry_MX_PCB_1.00u, F.Cu at (218.3, 267.7)
- added MX5: MX-NoLED, Switch_Keyboard_Cherry_MX:SW_Cherry_MX_PCB_1.25u, F.Cu at (11.3, 327.7)
- added MX50: MX-NoLED, Switch_Keyboard_Cherry_MX:SW_Cherry_MX_PCB_1.00u, F.Cu at (223.3, 287.7)
- added MX51: MX-NoLED, Switch_Keyboard_Cherry_MX:SW_Cherry_MX_PCB_1.00u, F.Cu at (233.3, 307.7)
- added MX52: MX-NoLED, Switch_Keyboard_Cherry_MX:SW_Cherry_MX_PCB_1.25u, F.Cu at (285.2, 327.7)
- added MX53: MX-NoLED, Switch_Keyboard_Cherry_MX:SW_Cherry_MX_PCB_1.00u, F.Cu at (228.3, 247.7)
- added MX54: MX-NoLED, Switch_Keyboard_Cherry_MX:SW_Cherry_MX_PCB_1.00u, F.Cu at (238.3, 267.7)
- added MX55: MX-NoLED, Switch_Keyboard_Cherry_MX:SW_Cherry_MX_PCB_1.00u, F.Cu at (243.3, 287.7)
- added MX56: MX-NoLED, Switch_Keyboard_Cherry_MX:SW_Cherry_MX_PCB_1.00u, F.Cu at (248.3, 247.7)
- added MX57: MX-NoLED, Switch_Keyboard_Cherry_MX:SW_Cherry_MX_PCB_1.00u, F.Cu at (258.3, 267.7)
- added MX58: MX-NoLED, Switch_Keyboard_Cherry_MX:SW_Cherry_MX_PCB_2.00u, F.Cu at (277.9, 247.7)
- added MX59: MX-NoLED, Switch_Keyboard_Cherry_MX:SW_Cherry_MX_PCB_1.50u, F.Cu at (282.9, 267.7)
- added MX6: MX-NoLED, Switch_Keyboard_Cherry_MX:SW_Cherry_MX_PCB_1.00u, F.Cu at (28.3, 247.7)
- added MX60: MX-NoLED, Switch_Keyboard_Cherry_MX:SW_Cherry_MX_PCB_2.25u, F.Cu at (275.8, 287.7)
- added MX61: MX-NoLED, Switch_Keyboard_Cherry_MX:SW_Cherry_MX_PCB_2.75u, F.Cu at (271.0, 307.7)
- added MX7: MX-NoLED, Switch_Keyboard_Cherry_MX:SW_Cherry_MX_PCB_1.00u, F.Cu at (38.3, 267.7)
- added MX8: MX-NoLED, Switch_Keyboard_Cherry_MX:SW_Cherry_MX_PCB_1.00u, F.Cu at (43.3, 287.7)
- added MX9: MX-NoLED, Switch_Keyboard_Cherry_MX:SW_Cherry_MX_PCB_1.00u, F.Cu at (53.3, 307.7)
- moved MH2 246.5 mm to (295.4, 235.3), turned to 180 degrees
- moved J2 242.5 mm to (292.9, 235.3), turned to 90 degrees
- moved MH1 229.0 mm to (295.4, 220.1), turned to 180 degrees
- moved J1 224.7 mm to (292.9, 220.1), turned to 90 degrees
- moved MH3 183.3 mm to (249.7, 235.3), turned to 180 degrees
- moved MH4 159.0 mm to (249.7, 220.1), turned to 180 degrees
Routing:
- net Row 4: track 0.00 -> 291.8 mm, vias 0 -> 12
- net Row 3: track 0.00 -> 279.1 mm, vias 0 -> 13
- net Row 2: track 0.00 -> 266.1 mm, vias 0 -> 14
- net Row 1: track 0.00 -> 249.3 mm, vias 0 -> 14
- net Row 5: track 0.00 -> 240.2 mm, vias 0 -> 8
- net Net-(D52-Pad2): track 0.00 -> 156.0 mm
- net Net-(D47-Pad2): track 0.00 -> 150.9 mm
- net Net-(D42-Pad2): track 0.00 -> 147.2 mm
- net Net-(D37-Pad2): track 0.00 -> 138.2 mm
- net Col 11: track 0.00 -> 134.4 mm
- net Net-(D10-Pad2): track 0.00 -> 130.5 mm
- net Net-(D61-Pad2): track 0.00 -> 128.0 mm
- net Net-(D15-Pad2): track 0.00 -> 123.8 mm
- net Net-(D24-Pad2): track 0.00 -> 119.3 mm
- net Col 9: track 0.00 -> 118.7 mm
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- added copper zone on B.Cu, net GND
Other:
- board size 48.3 x 17.8 mm -> 299.1 x 124.2 mm
