File: Keyboard Project V1/60 Percent Keyboard Project/60 Percent Keyboard Ardiuno Micro.kicad_pcb (KiCad board)
At the start: 2 copper layers, 299.1 x 124.2 mm, 129 parts, among them J1 Analog, J2 Digital

Commit message: Finally completed 1 versiongit add .!
Parts:
- removed J1: Analog, Connector_PinHeader_2.54mm:PinHeader_1x17_P2.54mm_Vertical
- removed J2: Digital, Connector_PinHeader_2.54mm:PinHeader_1x17_P2.54mm_Vertical
- removed MH1, MH2, MH3, MH4: MountingHole_1.2mm, Arduino_MountingHole:MountingHole_1.2mm
- added G***: LOGO, Graphics_or_Pictures:butterflies with color, F.Cu at (37.6, 285.3)
- A1, D1, D10, D11, D12, D13, D14, D15, D16, D17, D18, D19, D2, D20, D21, D22, D23, D24, D25, D26, D27, D28, D29, D3, D30, D31, D32, D33, D34, D35, D36, D37, D38, D39, D4, D40, D41, D42, D43, D44, D45, D46, D47, D48, D49, D5, D50, D51, D52, D53, D54, D55, D56, D57, D58, D59, D6, D60, D61, D7, D8, D9, MX1, MX10, MX11, MX12, MX13, MX14, MX15, MX16, MX17, MX18, MX19, MX2, MX20, MX21, MX22, MX23, MX24, MX25, MX26, MX27, MX28, MX29, MX3, MX30, MX31, MX32, MX33, MX34, MX35, MX36, MX37, MX38, MX39, MX4, MX40, MX41, MX42, MX43, MX44, MX45, MX46, MX47, MX48, MX49, MX5, MX50, MX51, MX52, MX53, MX54, MX55, MX56, MX57, MX58, MX59, MX6, MX60, MX61, MX7, MX8, MX9: moved to B.Cu
- moved D1 285.1 mm to (290.9, 223.4)
- moved MX1 279.1 mm to (287.9, 247.7), turned to 180 degrees
- moved D2 277.1 mm to (286.9, 223.4)
- moved MX5 274.1 mm to (285.4, 327.7), turned to 180 degrees
- moved MX52 273.7 mm to (11.5, 327.7), turned to 180 degrees
- moved MX2 270.1 mm to (283.4, 267.7), turned to 180 degrees
- moved MX59 269.1 mm to (13.8, 267.7), turned to 180 degrees
- moved D3 269.1 mm to (282.9, 223.4)
- moved MX3 265.1 mm to (280.9, 287.7), turned to 180 degrees
- moved D4 261.1 mm to (278.9, 223.4)
- moved MX58 259.1 mm to (18.8, 247.7), turned to 180 degrees
- moved MX4 255.1 mm to (275.9, 307.7), turned to 180 degrees
- moved MX60 254.9 mm to (20.9, 287.7), turned to 180 degrees
- moved D5 253.1 mm to (274.9, 223.4)
- moved MX61 245.2 mm to (25.7, 307.7), turned to 180 degrees
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Connections:
- A1 pad 27: +5V -> (no net)
- A1 pad 28: Net-(A1-Pad28) -> unconnected-(A1-Pad28)
- A1 pad 29: GND -> unconnected-(A1-Pad29)
- A1 pad 3: Net-(A1-Pad28) -> unconnected-(A1-Pad3)
- A1 pad 30: +5V -> (no net)
- A1 pad 4: GND -> unconnected-(A1-Pad4)
Routing:
- net Col 3: track 70.4 -> 404.3 mm, vias 0 -> 3
- net Col 1: track 91.1 -> 377.5 mm
- net Col 2: track 98.6 -> 368.5 mm, vias 0 -> 2
- net Col 4: track 70.4 -> 329.6 mm, vias 0 -> 2
- net Col 6: track 70.4 -> 283.6 mm
- net Col 5: track 99.7 -> 306.9 mm, vias 0 -> 2
- net Col 7: track 70.4 -> 263.6 mm
- net Col 8: track 116.9 -> 272.4 mm, vias 0 -> 2
- net Col 9: track 118.7 -> 246.0 mm, vias 0 -> 2
- net Col 10: track 117.1 -> 234.6 mm, vias 0 -> 2
- net Col 11: track 134.4 -> 238.7 mm, vias 0 -> 2
- net Col 12: track 46.2 -> 133.6 mm
- net Row 5: track 240.2 -> 306.1 mm, vias 8 -> 9
- net Col 14: track 67.0 -> 129.1 mm, vias 0 -> 2
- net Row 1: track 249.3 -> 308.7 mm
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- added copper zone on F.Cu, net unconnected-(A1-Pad29)
- removed copper zone on B.Cu, net GND
Other:
- outline, holes or cut-outs redrawn
- board text added: "Arty-Chan T-T"
- board text removed: "ICSP"
- board text removed: "USB Micro-B"
