File: Keyboard Project V3/65_percent_keyboard/65_percent_keyboard.kicad_sch (KiCad schematic)
At the start: 50 parts, among them SW1 SW_Push, U1 ATmega32A-P, U2 FT232RL, Y1 16MHz

Commit message: fixed most of the components
Parts:
- removed D10, D11, D12, D13, D14, D15, D16, D17, D7, D8, D9: SOD-123, Diode_SMD:D_SOD-123, symbol Device:D_Small
- removed MX10, MX11, MX12, MX13, MX14, MX15, MX16, MX17, MX7, MX8, MX9: MX-NoLED, MX_Alps_Hybrid:MX-1U-NoLED, symbol MX_Alps_Hybrid:MX-NoLED
- removed USB1: Molex-0548190589, random-keyboard-parts:Molex-0548190589, symbol random-keyboard-parts:Molex-0548190589
Connections:
- net COL3 is gone; now on net ROW0: U1.37 (PA3)
- net ROW0: no longer U1.36 (PA4)
- net ROW1: now also U1.36 (PA4); no longer U1.35 (PA5)
- net ROW2: no longer names the net of U1.34 (PA6)
- net ROW3: no longer names the net of U1.33 (PA7)
- net ROW4: no longer names the net of U1.1 (PB0)
Other:
- note added: "- Link 2"
- note added: "- Link 3"
- note added: "- Link 4"
- note added: "Christopher Morales (Arty-Chan)"
- note added: "Version 2: - Type C - No LED - No Encoder (Volumne Knob) - No Bluetooth Module"
- note removed: "Version 2: - Mirco USB - No Type C - No LED - No Encoder (Volumne Knob) - No Bluetooth Module"
